Commit message: better organization files update, arms poses parametrized in sim.launch

File: iliad/urdf/franka_robot.xacro (robot description, xacro)
@@ -2,5 +2,4 @@
 <robot xmlns:xacro="http://www.ros.org/wiki/xacro">
   <xacro:macro name="franka_robot" params="arm_id joint_limits">
-    <!-- Name of this panda -->
     <!-- Should a franka_gripper be mounted at the flange?" -->
     <xacro:arg name="hand" default="false" />
@@ -12,6 +11,6 @@
     <xacro:arg name="gazebo" default="true" />
     <xacro:include filename="$(find franka_description)/robots/common/utils.xacro" />
-    <xacro:include filename="$(find franka_description)/robots/common/franka_arm.xacro" />
-    <xacro:franka_arm arm_id="${arm_id}" safety_distance="0.03" gazebo="$(arg gazebo)" joint_limits="${joint_limits}" connected_to="robot_base_chapa" xyz='0.20 -0.15 0.05'/>
+    <xacro:include filename="$(find iliad)/urdf/franka_arm.xacro" />
+    <xacro:franka_arm arm_id="${arm_id}" safety_distance="0.03" gazebo="$(arg gazebo)" joint_limits="${joint_limits}" />
     <xacro:if value="$(arg hand)">
       <xacro:include filename="$(find franka_description)/robots/common/franka_hand.xacro"/>
@@ -30,11 +29,4 @@
       <xacro:arg name="xyz" default="0 0 0" />
       <xacro:arg name="rpy" default="0 0 0" />
-      <!-- Gazebo requires a joint to a link called "world" for statically mounted robots
-      <link name="world" />
-      <joint name="world_joint" type="fixed">
-        <origin xyz="$(arg xyz)" rpy="$(arg rpy)" />
-        <parent link="summit_xl_base_chapa" />
-        <child  link="$(arg arm_id)_link0" />
-      </joint>-->
         <!--
       <xacro:gazebo-joint joint="${arm_id}_joint1" transmission="hardware_interface/PositionJointInterface" />
@@ -59,10 +51,4 @@
       <xacro:gazebo-joint joint="${arm_id}_joint6" transmission="hardware_interface/EffortJointInterface" />
       <xacro:gazebo-joint joint="${arm_id}_joint7" transmission="hardware_interface/EffortJointInterface" />
-    <!--
-      <xacro:transmission-franka-state arm_id="${arm_id}" />
-      <xacro:transmission-franka-model arm_id="${arm_id}"
-         root="${arm_id}_joint1"
-         tip="${arm_id}_joint8"
-       />-->
       <xacro:if value="$(arg hand)">
         <xacro:gazebo-joint joint="${arm_id}_finger_joint1" transmission="hardware_interface/EffortJointInterface" />
@@ -72,13 +58,4 @@
         <xacro:gazebo-friction link="${arm_id}_rightfinger" mu="1.13" />
       </xacro:if>
-      <!--
-      <gazebo>
-        <plugin name="gazebo_ros_control" filename="libgazebo_ros_control.so">
-          <controlPeriod>0.001</controlPeriod>
-          <robotSimType>franka_gazebo/FrankaHWSim</robotSimType>
-        </plugin>
-        <self_collide>true</self_collide>
-      </gazebo>
-      -->
     </xacro:if>
   </xacro:macro>

File: iliad/urdf/iliad.urdf.xacro (robot description, xacro)
@@ -1,73 +1,32 @@
 <?xml version="1.0"?>
 <robot name="iliad" xmlns:xacro="http://wiki.ros.org/xacro">
-	<!-- *****************  Imported elements  ***************** -->
-	<!-- First we import all posible elements defined in the urdf.xacro files. All these elements are defined as macro:xacros -->
-	<!-- Import summit XL base elements and wheels -->
-	<xacro:include filename="$(find iliad)/urdf/summit_xls_base.urdf.xacro" />
-	<xacro:include filename="$(find iliad)/urdf/omni_wheel.urdf.xacro" />
-    <xacro:include filename="$(find summit_xl_description)/urdf/bases/summit_xl_base.gazebo.xacro" />
-	<xacro:property name="PI" value="3.1415926535897931"/>
-	<!-- Wheel parameters -->
-	<xacro:property name="wheel_offset_x" value="0.2225" />    <!-- x,y,z in translation from base_link to the center of the wheel -->
-	<xacro:property name="wheel_offset_y" value="0.2045" />
-	<xacro:property name="wheel_offset_z" value="0.0" />
-	<!-- Flag to select the high or low quality model -->
-    <xacro:property name="hq" value="true" />
-	<xacro:arg name="prefix" default="summit_xl_"/>
-	<xacro:arg name="ros_planar_move_plugin" default="true"/>
-	<xacro:arg name="ros_planar_move_plugin_force_based" default="true"/>
-	<xacro:arg name="gpu" default="true"/>
-    <xacro:macro name="summit_xl" params="prefix publish_bf hq">
-		<!-- Here we create the robot elements using the xacro:macros imported at the beggining of this file -->
-		<xacro:summit_xls_base prefix="$(arg prefix)" publish_bf="true" hq="${hq}" />
-		<xacro:omni_wheel prefix="$(arg prefix)front_right" parent="$(arg prefix)base_link" reflect="false" hq="${hq}">
-			<origin xyz="${wheel_offset_x} -${wheel_offset_y} ${wheel_offset_z}" rpy="0 0 0"/>
-		</xacro:omni_wheel>
-		<xacro:omni_wheel prefix="$(arg prefix)front_left" parent="$(arg prefix)base_link" reflect="true" hq="${hq}">
-			<origin xyz="${wheel_offset_x} ${wheel_offset_y} ${wheel_offset_z}" rpy="0 0 0"/>
-		</xacro:omni_wheel>
-		<xacro:omni_wheel prefix="$(arg prefix)back_left" parent="$(arg prefix)base_link" reflect="true" hq="${hq}">
-			<origin xyz="-${wheel_offset_x} ${wheel_offset_y} ${wheel_offset_z}" rpy="0 0 0"/>
-		</xacro:omni_wheel>
-		<xacro:omni_wheel prefix="$(arg prefix)back_right" parent="$(arg prefix)base_link" reflect="false" hq="${hq}">
-			<origin xyz="-${wheel_offset_x} -${wheel_offset_y} ${wheel_offset_z}" rpy="0 0 0"/>
-		</xacro:omni_wheel>
-    </xacro:macro>
-    <!-- Robot Assembling -->
-    <xacro:summit_xl prefix="$(arg prefix)" publish_bf="true" hq="true"/>
-    <!-- ********************************************************************************************************************************************* -->
-    <!-- ********************************************************************************************************************************************* -->
-    <!-- ********************************************************************************************************************************************* -->
-    <!-- Here I should add UR10e arm -->
+    <xacro:arg name="panda_base_x"     default="0"/>
+    <xacro:arg name="panda_base_y"     default="0"/>
+    <xacro:arg name="panda_base_z"     default="0"/>
+    <xacro:arg name="panda_base_roll"  default="0"/>
+    <xacro:arg name="panda_base_pitch" default="0"/>
+    <xacro:arg name="panda_base_yaw"   default="0"/>
+    <xacro:arg name="ur10e_base_x"     default="0"/>
+    <xacro:arg name="ur10e_base_y"     default="0"/>
+    <xacro:arg name="ur10e_base_z"     default="0"/>
+    <xacro:arg name="ur10e_base_roll"  default="0"/>
+    <xacro:arg name="ur10e_base_pitch" default="0"/>
+    <xacro:arg name="ur10e_base_yaw"   default="0"/>
+    <xacro:arg name="summit_prefix" default="summitxls_"/>
+    <xacro:arg name="ur10e_prefix"  default="ur10e_"/>
+    <xacro:arg name="panda_prefix"  default="panda"/>
+    <xacro:include filename="$(find iliad)/urdf/summit_macro.xacro"/>
     <xacro:include filename="$(find iliad)/urdf/ur_macro.xacro"/>
-    <xacro:arg name="robot_model" default="ur10e" />
-    <!--Parameter files -->
-    <xacro:arg name="joint_limit_params" default="$(find ur_description)/config/ur10e/joint_limits.yaml"/>
-    <xacro:arg name="kinematics_params" default="$(find ur_description)/config/ur10e/default_kinematics.yaml"/>
-    <xacro:arg name="physical_params" default="$(find ur_description)/config/ur10e/physical_parameters.yaml"/>
-    <xacro:arg name="visual_params" default="$(find ur_description)/config/ur10e/visual_parameters.yaml"/>
-    <!--Common parameters -->
-    <xacro:arg name="transmission_hw_interface" default="hardware_interface/EffortJointInterface" doc="The hardware_interface to expose for each joint in the simulated robot (one of: [PositionJointInterface, VelocityJointInterface, EffortJointInterface])"/>
-    <xacro:arg name="safety_limits" default="false" doc="If True, enable the safety limits controller"/>
-    <xacro:arg name="safety_pos_margin" default="0.15" doc="The lower/upper limits in the safety controller" />
-    <xacro:arg name="safety_k_position" default="20" doc="Used to set k position in the safety controller" />
-    <!-- Instantiate the Gazebo robot and pass it all the required arguments. -->
-    <xacro:ur_robot_gazebo
-        prefix="ur_"
-        joint_limits_parameters_file="$(arg joint_limit_params)"
-        kinematics_parameters_file="$(arg kinematics_params)"
-        physical_parameters_file="$(arg physical_params)"
-        visual_parameters_file="$(arg visual_params)"
-        transmission_hw_interface="$(arg transmission_hw_interface)"
-        safety_limits="$(arg safety_limits)"
-        safety_pos_margin="$(arg safety_pos_margin)"
-        safety_k_position="$(arg safety_k_position)"
-    />
-    <joint name="summit_tu_ur10e" type="fixed">
-        <parent link="robot_base_chapa"/>
-        <child link="ur_base_link"/>
-        <origin xyz="0.24 0.18 0" rpy="0 0 0"/>
+    <xacro:include filename="$(find iliad)/urdf/franka_robot.xacro"/>
+    <!-- Robot Assembling   -->
+    <xacro:summit_xls_macro prefix="$(arg summit_prefix)" publish_bf="true" hq="true"/>
+    <xacro:ur_robot_gazebo prefix="$(arg ur10e_prefix)"/>
+    <joint name="summit_to_ur10e" type="fixed">
+        <parent link="$(arg summit_prefix)base_chapa"/>
+        <child  link="$(arg ur10e_prefix)base_link"/>
+        <origin xyz="$(arg ur10e_base_x) $(arg ur10e_base_y) $(arg ur10e_base_z)"
+                rpy="$(arg ur10e_base_roll) $(arg ur10e_base_pitch) $(arg ur10e_base_yaw)"/>
     </joint>
-<!--
+    <!--
     <link name="tool0_controller"/>
     <joint name="tool_controller_fake_joint" type="fixed">
@@ -76,15 +35,13 @@
     <origin xyz="0 0 0" rpy="0 0 0"/>
     </joint>-->
+    <xacro:franka_robot arm_id="$(arg panda_prefix)" joint_limits="${xacro.load_yaml('$(find iliad)/robots/joint_limits.yaml')}"/>
+    <joint name="$summit_to_panda" type="fixed">
+        <parent link="$(arg summit_prefix)base_chapa"/>
+        <child  link="$(arg panda_prefix)_link0"/>
+        <origin xyz="$(arg panda_base_x) $(arg panda_base_y) $(arg panda_base_z)"
+                rpy="$(arg panda_base_roll) $(arg panda_base_pitch) $(arg panda_base_yaw)" />
+    </joint>
     <!-- ********************************************************************************************************************************************* -->
-    <!-- ********************************************************************************************************************************************* -->
-    <!-- ********************************************************************************************************************************************* -->
-   <!-- Here I should add Franka Panda arm
-   <xacro:panda connected_to="" xyz="" rpy="" />-->
-   <xacro:include filename="$(find iliad)/urdf/franka_robot.xacro"/>
-    <xacro:arg name="arm_id" default="panda" />
-    <xacro:franka_robot arm_id="$(arg arm_id)"
-                        joint_limits="${xacro.load_yaml('$(find iliad)/robots/joint_limits.yaml')}">
-    </xacro:franka_robot>
-   <!-- ROS Plugins -->
+    <!-- ROS Plugins -->
     <gazebo>
         <plugin name="ros_control" filename="libgazebo_ros_control.so">
@@ -96,7 +53,11 @@
         </plugin>
     </gazebo>
-     <!--
-   <xacro:if value="$(arg ros_planar_move_plugin)">
-	   <xacro:omni_steering prefix="$(arg prefix)" publish_tf="true" force_based="$(arg ros_planar_move_plugin_force_based)"/>
-   </xacro:if>-->
+    <xacro:include filename="$(find summit_xl_description)/urdf/bases/summit_xl_base.gazebo.xacro" />
+    <xacro:arg name="ros_planar_move_plugin" default="true"/>
+	<xacro:arg name="ros_planar_move_plugin_force_based" default="true"/>
+    <!-- <xacro:arg name="gpu" default="true"/>
+    <xacro:if value="$(arg ros_planar_move_plugin)">
+        <xacro:omni_steering prefix="$(arg summit_prefix)" publish_tf="true" force_based="$(arg ros_planar_move_plugin_force_based)"/>
+    </xacro:if>
+    -->
 </robot>

File: iliad/urdf/ur_macro.xacro (robot description, xacro)
@@ -32,11 +32,5 @@
   <!-- Definition of the main macro -->
   <xacro:macro name="ur_robot_gazebo" params="
-   prefix
-   joint_limits_parameters_file
-   kinematics_parameters_file
-   physical_parameters_file
-   visual_parameters_file
-   transmission_hw_interface:=hardware_interface/EffortJointInterface
-   safety_limits:=false safety_pos_margin:=0.15 safety_k_position:=20"
+   prefix"
   >
     <!--
@@ -47,4 +41,14 @@
     -->
   <xacro:include filename="$(find ur_description)/urdf/inc/ur_macro.xacro"/>
+    Parameter files -->
+    <xacro:property name="joint_limits_parameters_file" value="$(find ur_description)/config/ur10e/joint_limits.yaml"/>
+    <xacro:property name="kinematics_parameters_file" value="$(find ur_description)/config/ur10e/default_kinematics.yaml"/>
+    <xacro:property name="physical_parameters_file" value="$(find ur_description)/config/ur10e/physical_parameters.yaml"/>
+    <xacro:property name="visual_parameters_file" value="$(find ur_description)/config/ur10e/visual_parameters.yaml"/>
+    <!--Common parameters -->
+    <xacro:property name="transmission_hw_interface" value="hardware_interface/EffortJointInterface"/> <!--doc="The hardware_interface to expose for each joint in the simulated robot (one of: [PositionJointInterface, VelocityJointInterface, EffortJointInterface])"-->
+    <xacro:property name="safety_limits" value="false"/> <!--doc="If True, enable the safety limits controller"-->
+    <xacro:property name="safety_pos_margin" value="0.15"/> <!--doc="The lower/upper limits in the safety controller" -->
+    <xacro:property name="safety_k_position" value="20" /> <!--doc="Used to set k position in the safety controller"-->
     <!-- Instantiate model for the REAL robot. -->
     <xacro:ur_robot
