Commit message: Comments added and code cleared

File: iliad/urdf/armsBase.urdf.xacro (robot description, xacro)
@@ -1,4 +1,8 @@
 <?xml version="1.0"?>
 <robot xmlns:xacro="http://www.ros.org/wiki/xacro">
+<!-- This file create arms_base link to connect Franka and UR10e manipulator bases to Summit chassis.
+     The dimensions of collision box and mass are qualitatives.
+     The .stl mesh is designed based on the chosen configuration of the robot
+     -->
 <xacro:property name="arb_box_x" value="0.2"/>
 <xacro:property name="arb_box_y" value="0.57"/>

File: iliad/urdf/controlBoxes.urdf.xacro (robot description, xacro)
@@ -1,4 +1,7 @@
 <?xml version="1.0"?>
 <robot xmlns:xacro="http://www.ros.org/wiki/xacro">
+    <!-- This file create controller_unit link simulating the controller units of manipulators linked to the Summit chassis.
+     The dimensions of collision box are qualitatives, while the mass and the visual are referred to real control boxes.
+     -->
     <xacro:property name="ctr_box_x" value="0.25"/>
     <xacro:property name="ctr_box_y" value="0.46"/>

File: iliad/urdf/flange.urdf.xacro (robot description, xacro)
@@ -1,4 +1,8 @@
 <?xml version="1.0"?>
 <robot xmlns:xacro="http://www.ros.org/wiki/xacro">
+    <!-- This file create flange link between the last link of Franka manipulator and the IIT/Pisa SoftHand.
+         This link emulate the real configuration in CentroPiaggio laboratories for Franka manipulator.
+         The visuals, collisions and mass are qualitatives.
+     -->
     <xacro:property name="fl_box_x" value="0.10"/>
     <xacro:property name="fl_box_y" value="0.06"/>

File: iliad/urdf/omni_wheel.urdf.xacro (robot description, xacro)
@@ -72,17 +72,5 @@
       <kp value="10000000.0" />
       <kd value="1.0" />
-      <!--<fdir1 value="1 0 0"/>
-      <turnGravityOff>false</turnGravityOff>-->
     </gazebo>
-    <!--
-    <gazebo reference="${prefix}_wheel_link">
-		<mu1 value="200.0"/>
-		<mu2 value="100.0"/>
-		<kp value="10000000.0" />
-		<kd value="1.0" />
-		<fdir1 value="1 0 0"/>
-        <turnGravityOff>false</turnGravityOff>
-    </gazebo>
-    -->
   </xacro:macro>
 </robot>

File: iliad/urdf/velvet.urdf.xacro (robot description, xacro)
@@ -1,4 +1,8 @@
 <?xml version="1.0"?>
 <robot xmlns:xacro="http://www.ros.org/wiki/xacro">
+<!-- ************************** !! ****************************
+    This is the old file used in vito_robot project.
+    Please see velvet_new file with collision and inertial properties updated.
+-->
 <!-- conversions -->
 <!-- I couldn't make the simulation work with realistic values, so I tweaked the conversion values -->

File: iliad/urdf/velvet_new.urdf.xacro (robot description, xacro)
@@ -1,52 +1,55 @@
 <?xml version="1.0"?>
 <robot xmlns:xacro="http://www.ros.org/wiki/xacro">
-<xacro:property name="vel_box_x" value="0.14"/>
-<xacro:property name="vel_box_y" value="0.08"/>
-<xacro:property name="vel_box_z" value="0.28"/>
-<xacro:property name="vel_box_dim" value="${vel_box_x} ${vel_box_y} ${vel_box_z}"/>
-<xacro:property name="vel_mass" value="1"/>
-<xacro:macro name="velvet_macro" params="parent name *origin">
-    <joint name="${parent}_${name}" type="fixed">
-        <xacro:insert_block name="origin"/>
-        <parent link="${parent}"/>
-        <child link="${name}"/>
-    </joint>
-    <link name="${name}">
-        <visual>
-      <geometry>
-        <mesh filename="package://iliad/meshes/gazebo_assieme.stl"/>
-      </geometry>
-      <material name="green">
-          <color rgba="0 1 0 1"/>
-      </material>
-    </visual>
-    <inertial>
-        <origin xyz="0 0 0"/>
-        <mass value="${vel_mass}"/>
-        <inertia ixx="${vel_mass/12*(vel_box_y*vel_box_y+vel_box_z*vel_box_z)}" ixy="0.0" ixz="0.0" iyy="${vel_mass/12*(vel_box_x*vel_box_x+vel_box_z*vel_box_z)}" iyz="0.0" izz="${vel_mass/12*(vel_box_x*vel_box_x+vel_box_y*vel_box_y)}"/>
-    </inertial>
-    <collision>
-      <geometry>
-           <box size="${vel_box_dim}"/>
-      </geometry>
-      <origin rpy="0 0 0" xyz="0 0 0"/>
-    </collision>
-    </link>
-  <gazebo reference="${name}">
-     <!--<static>true</static> -->
-    <mu1 value="1.0"/>
-    <mu2 value="1.0"/>
-    <kp value="1e+13" />
-    <kd value="1.0" />
-    <collision>
-      <surface>
-        <contact>
-          <ode>
-            <min_depth>0.01</min_depth>
-          </ode>
-        </contact>
-      </surface>
-    </collision>
-  </gazebo>
-</xacro:macro>
+  <!-- This file create the velvet end effector after the last UR10e link.
+        This link is based on the real velvet tray in Centro Piaggio, already used in WRAPP-up project (vito-robot repository)
+    -->
+  <xacro:property name="vel_box_x" value="0.14"/>
+  <xacro:property name="vel_box_y" value="0.08"/>
+  <xacro:property name="vel_box_z" value="0.28"/>
+  <xacro:property name="vel_box_dim" value="${vel_box_x} ${vel_box_y} ${vel_box_z}"/>
+  <xacro:property name="vel_mass" value="1"/>
+  <xacro:macro name="velvet_macro" params="parent name *origin">
+      <joint name="${parent}_${name}" type="fixed">
+          <xacro:insert_block name="origin"/>
+          <parent link="${parent}"/>
+          <child link="${name}"/>
+      </joint>
+      <link name="${name}">
+          <visual>
+        <geometry>
+          <mesh filename="package://iliad/meshes/gazebo_assieme.stl"/>
+        </geometry>
+        <material name="green">
+            <color rgba="0 1 0 1"/>
+        </material>
+      </visual>
+      <inertial>
+          <origin xyz="0 0 0"/>
+          <mass value="${vel_mass}"/>
+          <inertia ixx="${vel_mass/12*(vel_box_y*vel_box_y+vel_box_z*vel_box_z)}" ixy="0.0" ixz="0.0" iyy="${vel_mass/12*(vel_box_x*vel_box_x+vel_box_z*vel_box_z)}" iyz="0.0" izz="${vel_mass/12*(vel_box_x*vel_box_x+vel_box_y*vel_box_y)}"/>
+      </inertial>
+      <collision>
+        <geometry>
+            <box size="${vel_box_dim}"/>
+        </geometry>
+        <origin rpy="0 0 0" xyz="0 0 0"/>
+      </collision>
+      </link>
+    <gazebo reference="${name}">
+      <!--<static>true</static> -->
+      <mu1 value="1.0"/>                    <!--change this to get more real simulation in gazebo-->
+      <mu2 value="1.0"/>
+      <kp value="1e+13" />
+      <kd value="1.0" />
+      <collision>
+        <surface>
+          <contact>
+            <ode>
+              <min_depth>0.01</min_depth>   <!--change this to get more real simulation in gazebo-->
+            </ode>
+          </contact>
+        </surface>
+      </collision>
+    </gazebo>
+  </xacro:macro>
 </robot>
