Commit message: summit & diff.drive ok

File: iliad/urdf/iliad.urdf.xacro (robot description, xacro)
@@ -35,8 +35,17 @@
    </xacro:macro>
    <xacro:summit_xl prefix="$(arg prefix)" publish_bf="true" hq="true"/>
-   <!---->
-   <xacro:ros_control/>
+   <!-- ROS Plugins -->
+    <gazebo>
+        <plugin name="ros_control" filename="libgazebo_ros_control.so">
+            <robotParam>robot_description</robotParam>
+            <controlPeriod>0.001</controlPeriod>
+            <robotSimType>gazebo_ros_control/DefaultRobotHWSim</robotSimType>
+            <legacyModeNS>true</legacyModeNS>
+        </plugin>
+    </gazebo>
+   <!--
    <xacro:if value="$(arg ros_planar_move_plugin)">
 	   <xacro:omni_steering prefix="$(arg prefix)" publish_tf="true" force_based="$(arg ros_planar_move_plugin_force_based)"/>
    </xacro:if>
+   -->
 </robot>

File: iliad/urdf/omni_wheel.urdf.xacro (robot description, xacro)
@@ -68,6 +68,6 @@
     </transmission>
     <gazebo reference="${prefix}_wheel_link">
-		<mu1 value="0.0"/>
-		<mu2 value="0.0"/>
+		<mu1 value="1.0"/>
+		<mu2 value="1.0"/>
 		<kp value="10000000.0" />
 		<kd value="1.0" />
@@ -75,4 +75,14 @@
         <turnGravityOff>false</turnGravityOff>
     </gazebo>
+    <!--
+    <gazebo reference="${prefix}_wheel_link">
+		<mu1 value="200.0"/>
+		<mu2 value="100.0"/>
+		<kp value="10000000.0" />
+		<kd value="1.0" />
+		<fdir1 value="1 0 0"/>
+        <turnGravityOff>false</turnGravityOff>
+    </gazebo>
+    -->
   </xacro:macro>
 </robot>

File: iliad/urdf/summit_xl_base.gazebo.xacro (robot description, xacro)
@@ -1,15 +1,13 @@
 <?xml version="1.0"?>
 <robot xmlns:xacro="http://wiki.ros.org/xacro">
-  <!-- ros control plugin -->
-  <xacro:macro name="ros_control">
+  <!-- ros control plugin
     <gazebo>
-      <plugin name="ros_control" filename="libgazebo_ros_control.so">
-		    <robotParam>robot_description</robotParam>
-        <controlPeriod>0.001</controlPeriod>
-	      <robotSimType>gazebo_ros_control/DefaultRobotHWSim</robotSimType>
-		    <legacyModeNS>true</legacyModeNS>
-      </plugin>
-    </gazebo>
-	</xacro:macro>
+        <plugin name="ros_control" filename="libgazebo_ros_control.so">
+            <robotParam>robot_description</robotParam>
+            <controlPeriod>0.001</controlPeriod>
+            <robotSimType>gazebo_ros_control/DefaultRobotHWSim</robotSimType>
+            <legacyModeNS>true</legacyModeNS>
+        </plugin>
+    </gazebo>-->
 	<!-- skid steering plugin -->
 	<xacro:macro name="skid_steering" params="prefix publish_tf">

Commit message: UR10e added with controllers !

File: iliad/urdf/iliad.urdf.xacro (robot description, xacro)
@@ -33,10 +33,57 @@
 			<origin xyz="-${wheel_offset_x} -${wheel_offset_y} ${wheel_offset_z}" rpy="0 0 0"/>
 		</xacro:omni_wheel>
-   </xacro:macro>
-   <xacro:summit_xl prefix="$(arg prefix)" publish_bf="true" hq="true"/>
+    </xacro:macro>
+    <!-- Robot Assembling -->
+    <xacro:summit_xl prefix="$(arg prefix)" publish_bf="true" hq="true"/>
+    <!-- ********************************************************************************************************************************************* -->
+    <!-- ********************************************************************************************************************************************* -->
+    <!-- ********************************************************************************************************************************************* -->
+    <!-- Here I should add UR10e arm -->
+    <xacro:include filename="$(find iliad)/urdf/ur_macro.xacro"/>
+    <xacro:arg name="robot_model" default="ur10e" />
+    <!--Parameter files -->
+    <xacro:arg name="joint_limit_params" default="$(find ur_description)/config/ur10e/joint_limits.yaml"/>
+    <xacro:arg name="kinematics_params" default="$(find ur_description)/config/ur10e/default_kinematics.yaml"/>
+    <xacro:arg name="physical_params" default="$(find ur_description)/config/ur10e/physical_parameters.yaml"/>
+    <xacro:arg name="visual_params" default="$(find ur_description)/config/ur10e/visual_parameters.yaml"/>
+    <!--Common parameters -->
+    <xacro:arg name="transmission_hw_interface" default="hardware_interface/EffortJointInterface" doc="The hardware_interface to expose for each joint in the simulated robot (one of: [PositionJointInterface, VelocityJointInterface, EffortJointInterface])"/>
+    <xacro:arg name="safety_limits" default="false" doc="If True, enable the safety limits controller"/>
+    <xacro:arg name="safety_pos_margin" default="0.15" doc="The lower/upper limits in the safety controller" />
+    <xacro:arg name="safety_k_position" default="20" doc="Used to set k position in the safety controller" />
+    <!-- Instantiate the Gazebo robot and pass it all the required arguments. -->
+    <xacro:ur_robot_gazebo
+        prefix="ur_"
+        joint_limits_parameters_file="$(arg joint_limit_params)"
+        kinematics_parameters_file="$(arg kinematics_params)"
+        physical_parameters_file="$(arg physical_params)"
+        visual_parameters_file="$(arg visual_params)"
+        transmission_hw_interface="$(arg transmission_hw_interface)"
+        safety_limits="$(arg safety_limits)"
+        safety_pos_margin="$(arg safety_pos_margin)"
+        safety_k_position="$(arg safety_k_position)"
+    />
+    <joint name="summit_tu_ur10e" type="fixed">
+    <parent link="robot_base_chapa"/>
+    <child link="ur_base_link"/>
+    <origin xyz="0.24 0.18 0" rpy="0 0 0"/>
+    </joint>
+<!--
+    <link name="tool0_controller"/>
+    <joint name="tool_controller_fake_joint" type="fixed">
+    <parent link="tool0"/>
+    <child link="tool0_controller"/>
+    <origin xyz="0 0 0" rpy="0 0 0"/>
+    </joint>-->
+    <!-- ********************************************************************************************************************************************* -->
+    <!-- ********************************************************************************************************************************************* -->
+    <!-- ********************************************************************************************************************************************* -->
+   <!-- Here I should add Franka Panda arm
+   <xacro:panda connected_to="" xyz="" rpy="" />-->
    <!-- ROS Plugins -->
     <gazebo>
         <plugin name="ros_control" filename="libgazebo_ros_control.so">
             <robotParam>robot_description</robotParam>
+            <robotNamespace>/</robotNamespace>
             <controlPeriod>0.001</controlPeriod>
             <robotSimType>gazebo_ros_control/DefaultRobotHWSim</robotSimType>
@@ -44,5 +91,4 @@
         </plugin>
     </gazebo>
-   <!---->
    <xacro:if value="$(arg ros_planar_move_plugin)">
 	   <xacro:omni_steering prefix="$(arg prefix)" publish_tf="true" force_based="$(arg ros_planar_move_plugin_force_based)"/>

Commit message: Franka Arm works

File: iliad/urdf/iliad.urdf.xacro (robot description, xacro)
@@ -65,7 +65,7 @@
     />
     <joint name="summit_tu_ur10e" type="fixed">
-    <parent link="robot_base_chapa"/>
-    <child link="ur_base_link"/>
-    <origin xyz="0.24 0.18 0" rpy="0 0 0"/>
+        <parent link="robot_base_chapa"/>
+        <child link="ur_base_link"/>
+        <origin xyz="0.24 0.18 0" rpy="0 0 0"/>
     </joint>
 <!--
@@ -81,4 +81,9 @@
    <!-- Here I should add Franka Panda arm
    <xacro:panda connected_to="" xyz="" rpy="" />-->
+   <xacro:include filename="$(find iliad)/urdf/franka_robot.xacro"/>
+    <xacro:arg name="arm_id" default="panda" />
+    <xacro:franka_robot arm_id="$(arg arm_id)"
+                        joint_limits="${xacro.load_yaml('$(find iliad)/robots/joint_limits.yaml')}">
+    </xacro:franka_robot>
    <!-- ROS Plugins -->
     <gazebo>
@@ -91,6 +96,7 @@
         </plugin>
     </gazebo>
+     <!--
    <xacro:if value="$(arg ros_planar_move_plugin)">
 	   <xacro:omni_steering prefix="$(arg prefix)" publish_tf="true" force_based="$(arg ros_planar_move_plugin_force_based)"/>
-   </xacro:if>
+   </xacro:if>-->
 </robot>

Commit message: add controller unit box

File: iliad/urdf/iliad.urdf.xacro (robot description, xacro)
@@ -42,4 +42,30 @@
                 rpy="$(arg panda_base_roll) $(arg panda_base_pitch) $(arg panda_base_yaw)" />
     </joint>
+    <link name="controller_unit">
+        <visual>
+            <geometry>
+                <box size="0.2 0.4 0.3"/>
+            </geometry>
+            <origin rpy="0 0 0" xyz="0 0 0"/>
+            <material name="white">
+                <color rgba="0.5 0.5 0.5 1"/>
+            </material>
+        </visual>
+        <collision>
+            <geometry>
+                <box size="0.2 0.4 0.30"/>
+            </geometry>
+            <origin rpy="0 0 0" xyz="0 0 0"/>
+        </collision>
+        <inertial>
+            <mass value="20"/>
+            <inertia ixx="1.0" ixy="0.0" ixz="0.0" iyy="1.0" iyz="0.0" izz="1.0"/>
+        </inertial>
+    </link>
+    <joint name="summit_to_controller_unit" type="fixed">
+        <parent link="$(arg summit_prefix)base_chapa"/>
+        <child link="controller_unit"/>
+        <origin xyz="-0.25 0 0.15"/>
+    </joint>
     <!-- ********************************************************************************************************************************************* -->
     <!-- ROS Plugins -->

Commit message: add new stl filles and better organization

File: iliad/urdf/iliad.urdf.xacro (robot description, xacro)
@@ -28,11 +28,9 @@
                 rpy="$(arg ur10e_base_roll) $(arg ur10e_base_pitch) $(arg ur10e_base_yaw)"/>
     </joint>
-    <!--
-    <link name="tool0_controller"/>
-    <joint name="tool_controller_fake_joint" type="fixed">
-    <parent link="tool0"/>
-    <child link="tool0_controller"/>
-    <origin xyz="0 0 0" rpy="0 0 0"/>
-    </joint>-->
+     <!---->
+   <xacro:include filename="$(find iliad)/urdf/velvet.urdf.xacro"/>
+    <xacro:model_velvet parent="ur10e_tool0" name="velvet">
+        <origin xyz="0 0 0.14" rpy="0 0 0"/>
+    </xacro:model_velvet>
     <xacro:franka_robot arm_id="$(arg panda_prefix)" joint_limits="${xacro.load_yaml('$(find iliad)/robots/joint_limits.yaml')}"/>
     <joint name="$summit_to_panda" type="fixed">
@@ -42,4 +40,41 @@
                 rpy="$(arg panda_base_roll) $(arg panda_base_pitch) $(arg panda_base_yaw)" />
     </joint>
+    <!--
+    <xacro:include filename="$(find softhands_description)/urdf/softhands.xacro"/>
+    <xacro:softhands type="right"
+        version = "v1.0_simple"
+        parent = "$(arg panda_prefix)_link8"
+        position ="0.05 -0.05 0.04"
+        orientation ="0 -1.57 2.355"
+        operation_mode = "0"
+        translation="0.0">
+    </xacro:softhands>
+    <link name="flange">
+        <visual>
+            <geometry>
+                <box size="0.10 0.06 0.08"/>
+            </geometry>
+            <origin rpy="0 0 0" xyz="0.02 0 0"/>
+            <material name="grey">
+                <color rgba="0.5 0.5 0.5 1"/>
+            </material>
+        </visual>
+        <collision>
+            <geometry>
+                <box size="0.10 0.06 0.08"/>
+            </geometry>
+            <origin rpy="0 0 0" xyz="0.02 0 0"/>
+        </collision>
+        <inertial>
+            <mass value="0.300"/>
+            <inertia ixx="0.00025" ixy="0.0" ixz="0.0" iyy="0.00041" iyz="0.0" izz="0.00034"/>
+        </inertial>
+    </link>
+    <joint name="panda_link8_to_hand" type="fixed">
+        <parent link="$(arg panda_prefix)_link8"/>
+        <child link="flange"/>
+        <origin rpy="0 0 -0.785" xyz="0 0 0.04"/>
+    </joint>
+    -->
     <link name="controller_unit">
         <visual>
@@ -48,5 +83,5 @@
             </geometry>
             <origin rpy="0 0 0" xyz="0 0 0"/>
-            <material name="white">
+            <material name="grey">
                 <color rgba="0.5 0.5 0.5 1"/>
             </material>
@@ -60,5 +95,5 @@
         <inertial>
             <mass value="20"/>
-            <inertia ixx="1.0" ixy="0.0" ixz="0.0" iyy="1.0" iyz="0.0" izz="1.0"/>
+            <inertia ixx="0.41666667" ixy="0.0" ixz="0.0" iyy="0.21666667" iyz="0.0" izz="0.33333333"/>
         </inertial>
     </link>
@@ -68,5 +103,5 @@
         <origin xyz="-0.25 0 0.15"/>
     </joint>
-    <!-- ********************************************************************************************************************************************* -->
+     <!--********************************************************************************************************************************************* -->
     <!-- ROS Plugins -->
     <gazebo>

Commit message: Arms plate mesh added

File: iliad/urdf/iliad.urdf.xacro (robot description, xacro)
@@ -40,6 +40,6 @@
                 rpy="$(arg panda_base_roll) $(arg panda_base_pitch) $(arg panda_base_yaw)" />
     </joint>
-    <!--
     <xacro:include filename="$(find softhands_description)/urdf/softhands.xacro"/>
+    <!---->
     <xacro:softhands type="right"
         version = "v1.0_simple"
@@ -76,5 +76,5 @@
         <origin rpy="0 0 -0.785" xyz="0 0 0.04"/>
     </joint>
-    -->
+    <!---->
     <link name="controller_unit">
         <visual>
@@ -103,4 +103,26 @@
         <origin xyz="-0.25 0 0.15"/>
     </joint>
+    <material name="steel">
+        <color rgba="0 0 0 1.0"/> <!-- rviz green color -->
+    </material>
+    <link name="arms_base">
+        <visual>
+            <geometry>
+                <mesh filename="package://iliad/meshes/arm_base.stl"/>
+            </geometry>
+            <material name="steel"/>
+        </visual>
+    </link>
+    <gazebo reference="arms_base">
+        <material>Gazebo/Grey</material>
+    </gazebo>
+    <gazebo reference="controller_unit">
+        <material>Gazebo/Grey</material>
+    </gazebo>
+    <joint name="summit_to_arms_base" type="fixed">
+        <parent link="$(arg summit_prefix)base_chapa"/>
+        <child link="arms_base"/>
+        <origin xyz="0.135 0.410 0" rpy="0 0 -1.57079632679"/>
+    </joint>
      <!--********************************************************************************************************************************************* -->
     <!-- ROS Plugins -->

File: iliad/urdf/velvet.urdf.xacro (robot description, xacro)
@@ -39,6 +39,6 @@
   <gazebo reference="${name}_link">
      <!--<static>true</static> -->
-    <mu1 value="10000000.0"/>
-    <mu2 value="10000000.0"/>
+    <mu1 value="1.0"/>
+    <mu2 value="1.0"/>
     <kp value="1e+13" />
     <kd value="1.0" />

Commit message: add control boxes .stl and create a new custom world for gazebo

File: iliad/urdf/iliad.urdf.xacro (robot description, xacro)
@@ -21,4 +21,5 @@
     <!-- Robot Assembling   -->
     <xacro:summit_xls_macro prefix="$(arg summit_prefix)" publish_bf="true" hq="true"/>
+ <!---->
     <xacro:ur_robot_gazebo prefix="$(arg ur10e_prefix)"/>
     <joint name="summit_to_ur10e" type="fixed">
@@ -28,5 +29,4 @@
                 rpy="$(arg ur10e_base_roll) $(arg ur10e_base_pitch) $(arg ur10e_base_yaw)"/>
     </joint>
-     <!---->
    <xacro:include filename="$(find iliad)/urdf/velvet.urdf.xacro"/>
     <xacro:model_velvet parent="ur10e_tool0" name="velvet">
@@ -41,5 +41,4 @@
     </joint>
     <xacro:include filename="$(find softhands_description)/urdf/softhands.xacro"/>
-    <!---->
     <xacro:softhands type="right"
         version = "v1.0_simple"
@@ -76,11 +75,10 @@
         <origin rpy="0 0 -0.785" xyz="0 0 0.04"/>
     </joint>
-    <!---->
     <link name="controller_unit">
         <visual>
             <geometry>
-                <box size="0.2 0.4 0.3"/>
-            </geometry>
-            <origin rpy="0 0 0" xyz="0 0 0"/>
+                <mesh filename="package://iliad/meshes/controller_boxes.stl"/>
+            </geometry>
+            <origin rpy="0 0 0" xyz="-0.1715 -0.2415 0"/>
             <material name="grey">
                 <color rgba="0.5 0.5 0.5 1"/>
@@ -89,11 +87,11 @@
         <collision>
             <geometry>
-                <box size="0.2 0.4 0.30"/>
-            </geometry>
-            <origin rpy="0 0 0" xyz="0 0 0"/>
-        </collision>
-        <inertial>
-            <mass value="20"/>
-            <inertia ixx="0.41666667" ixy="0.0" ixz="0.0" iyy="0.21666667" iyz="0.0" izz="0.33333333"/>
+                <mesh filename="package://iliad/meshes/controller_boxes.stl"/>
+            </geometry>
+            <origin rpy="0 0 0" xyz="-0.1715 -0.2415 0"/>
+        </collision>
+        <inertial>
+            <mass value="12"/>   <!-- franka 7kg, ur10e 5kg-->
+            <inertia ixx="0.2741" ixy="0.0" ixz="0.0" iyy="0.125" iyz="0.0" izz="0.2741"/>
         </inertial>
     </link>
@@ -101,5 +99,57 @@
         <parent link="$(arg summit_prefix)base_chapa"/>
         <child link="controller_unit"/>
-        <origin xyz="-0.25 0 0.15"/>
+        <origin xyz="-0.175 0 0"/>
+    </joint>
+    <link name="franka_controller_unit_plate">
+        <visual>
+            <geometry>
+                <mesh filename="package://iliad/meshes/franka_controller_box_plate.stl"/>
+            </geometry>
+            <origin rpy="0 0 0" xyz="-0.0175 -0.19 0"/>
+            <material name="grey">
+                <color rgba="1 1 1 1"/>
+            </material>
+        </visual>
+        <collision>
+            <geometry>
+                <mesh filename="package://iliad/meshes/franka_controller_box_plate.stl"/>
+            </geometry>
+            <origin rpy="0 0 0" xyz="-0.0175 -0.19 0"/>
+        </collision>
+        <inertial>
+            <mass value="0"/>
+            <inertia ixx="0.0" ixy="0.0" ixz="0.0" iyy="0.0" iyz="0.0" izz="0.0"/>
+        </inertial>
+    </link>
+    <joint name="controller_unit_TO_franka_plate" type="fixed">
+        <parent link="$(arg summit_prefix)base_chapa"/>
+        <child link="franka_controller_unit_plate"/>
+        <origin xyz="-0.259 0 0.351"/>
+    </joint>
+    <link name="ur_controller_unit_plate">
+        <visual>
+            <geometry>
+                <mesh filename="package://iliad/meshes/ur_controller_box_plate.stl"/>
+            </geometry>
+            <origin rpy="0 0 0" xyz="-0.0175 -0.19 0"/>
+            <material name="grey">
+                <color rgba="1 1 1 1"/>
+            </material>
+        </visual>
+        <collision>
+            <geometry>
+                <mesh filename="package://iliad/meshes/ur_controller_box_plate.stl"/>
+            </geometry>
+            <origin rpy="0 0 0" xyz="-0.0175 -0.19 0"/>
+        </collision>
+        <inertial>
+            <mass value="0"/>
+            <inertia ixx="0.0" ixy="0.0" ixz="0.0" iyy="0.0" iyz="0.0" izz="0.0"/>
+        </inertial>
+    </link>
+    <joint name="controller_unit_TO_ur_plate" type="fixed">
+        <parent link="$(arg summit_prefix)base_chapa"/>
+        <child link="ur_controller_unit_plate"/>
+        <origin xyz="-0.1305 0 0.164"/>
     </joint>
     <material name="steel">
@@ -113,4 +163,13 @@
             <material name="steel"/>
         </visual>
+        <collision>
+            <geometry>
+                <mesh filename="package://iliad/meshes/arm_base.stl"/>
+            </geometry>
+        </collision>
+        <inertial>
+            <mass value="2"/>   <!-- -->
+            <inertia ixx="0.2741" ixy="0.0" ixz="0.0" iyy="0.125" iyz="0.0" izz="0.2741"/>
+        </inertial>
     </link>
     <gazebo reference="arms_base">
@@ -119,4 +178,11 @@
     <gazebo reference="controller_unit">
         <material>Gazebo/Grey</material>
+    </gazebo>
+    <!---->
+    <gazebo reference="franka_controller_unit_plate">
+        <material>Gazebo/Black</material>
+    </gazebo>
+    <gazebo reference="ur_controller_unit_plate">
+        <material>Gazebo/Black</material>
     </gazebo>
     <joint name="summit_to_arms_base" type="fixed">

Commit message: update new velvet file

File: iliad/urdf/iliad.urdf.xacro (robot description, xacro)
@@ -29,5 +29,5 @@
                 rpy="$(arg ur10e_base_roll) $(arg ur10e_base_pitch) $(arg ur10e_base_yaw)"/>
     </joint>
-   <xacro:include filename="$(find iliad)/urdf/velvet.urdf.xacro"/>
+     <xacro:include filename="$(find iliad)/urdf/velvet_new.urdf.xacro"/>
     <xacro:model_velvet parent="ur10e_tool0" name="velvet">
         <origin xyz="0 0 0.14" rpy="0 0 0"/>
@@ -49,5 +49,5 @@
         translation="0.0">
     </xacro:softhands>
-    <link name="flange">
+  <link name="flange">
         <visual>
             <geometry>
@@ -68,4 +68,5 @@
             <mass value="0.300"/>
             <inertia ixx="0.00025" ixy="0.0" ixz="0.0" iyy="0.00041" iyz="0.0" izz="0.00034"/>
+            <origin rpy="0 0 0" xyz="0.02 0 0"/>
         </inertial>
     </link>
@@ -94,4 +95,5 @@
             <mass value="12"/>   <!-- franka 7kg, ur10e 5kg-->
             <inertia ixx="0.2741" ixy="0.0" ixz="0.0" iyy="0.125" iyz="0.0" izz="0.2741"/>
+            <origin rpy="0 0 0" xyz="0 0 0.13"/>
         </inertial>
     </link>
