Commit message: better code organization...

File: iliad/urdf/iliad.urdf.xacro (robot description, xacro)
@@ -19,7 +19,27 @@
     <xacro:include filename="$(find iliad)/urdf/ur_macro.xacro"/>
     <xacro:include filename="$(find iliad)/urdf/franka_robot.xacro"/>
+    <xacro:include filename="$(find iliad)/urdf/velvet_new.urdf.xacro"/>
+    <xacro:include filename="$(find softhands_description)/urdf/softhands.xacro"/>
+    <xacro:include filename="$(find iliad)/urdf/controlBoxes.urdf.xacro"/>
+    <xacro:include filename="$(find iliad)/urdf/armsBase.urdf.xacro"/>
+    <xacro:include filename="$(find iliad)/urdf/flange.urdf.xacro"/>
     <!-- Robot Assembling   -->
+    <!-- The ILIAD Robot is composed by:
+            - Summit XLS Steel
+            - UR10e Manipulator
+            - Franka Emika Panda Simulator
+            - Controller Boxes of manipulators
+            - A steel plate to connect Summit XLS to each manipulator
+            - A Customized velvet tray (UR10e end effector)
+            - A SoftHand (Franka end effector)
+            - A flange to connect the last Franka's link to the Softhand
+    -->
     <xacro:summit_xls_macro prefix="$(arg summit_prefix)" publish_bf="true" hq="true"/>
- <!---->
+    <xacro:controlBoxes_macro parent="$(arg summit_prefix)base_chapa" name="controller_unit">
+        <origin rpy="0 0 0" xyz="-0.175 0 0"/>
+    </xacro:controlBoxes_macro>
+    <xacro:armsBase_macro parent="$(arg summit_prefix)base_chapa" name="arms_base">
+        <origin xyz="0.270 0 0" rpy="0 0 0"/>
+    </xacro:armsBase_macro>
     <xacro:ur_robot_gazebo prefix="$(arg ur10e_prefix)"/>
     <joint name="summit_to_ur10e" type="fixed">
@@ -29,8 +49,7 @@
                 rpy="$(arg ur10e_base_roll) $(arg ur10e_base_pitch) $(arg ur10e_base_yaw)"/>
     </joint>
-     <xacro:include filename="$(find iliad)/urdf/velvet_new.urdf.xacro"/>
-    <xacro:model_velvet parent="ur10e_tool0" name="velvet">
+    <xacro:velvet_macro parent="ur10e_tool0" name="velvet">
         <origin xyz="0 0 0.14" rpy="0 0 0"/>
-    </xacro:model_velvet>
+    </xacro:velvet_macro>
     <xacro:franka_robot arm_id="$(arg panda_prefix)" joint_limits="${xacro.load_yaml('$(find iliad)/robots/joint_limits.yaml')}"/>
     <joint name="$summit_to_panda" type="fixed">
@@ -40,5 +59,7 @@
                 rpy="$(arg panda_base_roll) $(arg panda_base_pitch) $(arg panda_base_yaw)" />
     </joint>
-    <xacro:include filename="$(find softhands_description)/urdf/softhands.xacro"/>
+    <xacro:flange_macro parent="$(arg panda_prefix)_link8" name="flange">
+        <origin rpy="0 0 -0.785" xyz="0 0 0.04"/>
+    </xacro:flange_macro>
     <xacro:softhands type="right"
         version = "v1.0_simple"
@@ -49,149 +70,5 @@
         translation="0.0">
     </xacro:softhands>
-  <link name="flange">
-        <visual>
-            <geometry>
-                <box size="0.10 0.06 0.08"/>
-            </geometry>
-            <origin rpy="0 0 0" xyz="0.02 0 0"/>
-            <material name="grey">
-                <color rgba="0.5 0.5 0.5 1"/>
-            </material>
-        </visual>
-        <collision>
-            <geometry>
-                <box size="0.10 0.06 0.08"/>
-            </geometry>
-            <origin rpy="0 0 0" xyz="0.02 0 0"/>
-        </collision>
-        <inertial>
-            <mass value="0.300"/>
-            <inertia ixx="0.00025" ixy="0.0" ixz="0.0" iyy="0.00041" iyz="0.0" izz="0.00034"/>
-            <origin rpy="0 0 0" xyz="0.02 0 0"/>
-        </inertial>
-    </link>
-    <joint name="panda_link8_to_hand" type="fixed">
-        <parent link="$(arg panda_prefix)_link8"/>
-        <child link="flange"/>
-        <origin rpy="0 0 -0.785" xyz="0 0 0.04"/>
-    </joint>
-    <link name="controller_unit">
-        <visual>
-            <geometry>
-                <mesh filename="package://iliad/meshes/controller_boxes.stl"/>
-            </geometry>
-            <origin rpy="0 0 0" xyz="-0.1715 -0.2415 0"/>
-            <material name="grey">
-                <color rgba="0.5 0.5 0.5 1"/>
-            </material>
-        </visual>
-        <collision>
-            <geometry>
-                <mesh filename="package://iliad/meshes/controller_boxes.stl"/>
-            </geometry>
-            <origin rpy="0 0 0" xyz="-0.1715 -0.2415 0"/>
-        </collision>
-        <inertial>
-            <mass value="12"/>   <!-- franka 7kg, ur10e 5kg-->
-            <inertia ixx="0.2741" ixy="0.0" ixz="0.0" iyy="0.125" iyz="0.0" izz="0.2741"/>
-            <origin rpy="0 0 0" xyz="0 0 0.13"/>
-        </inertial>
-    </link>
-    <joint name="summit_to_controller_unit" type="fixed">
-        <parent link="$(arg summit_prefix)base_chapa"/>
-        <child link="controller_unit"/>
-        <origin xyz="-0.175 0 0"/>
-    </joint>
-    <link name="franka_controller_unit_plate">
-        <visual>
-            <geometry>
-                <mesh filename="package://iliad/meshes/franka_controller_box_plate.stl"/>
-            </geometry>
-            <origin rpy="0 0 0" xyz="-0.0175 -0.19 0"/>
-            <material name="grey">
-                <color rgba="1 1 1 1"/>
-            </material>
-        </visual>
-        <collision>
-            <geometry>
-                <mesh filename="package://iliad/meshes/franka_controller_box_plate.stl"/>
-            </geometry>
-            <origin rpy="0 0 0" xyz="-0.0175 -0.19 0"/>
-        </collision>
-        <inertial>
-            <mass value="0"/>
-            <inertia ixx="0.0" ixy="0.0" ixz="0.0" iyy="0.0" iyz="0.0" izz="0.0"/>
-        </inertial>
-    </link>
-    <joint name="controller_unit_TO_franka_plate" type="fixed">
-        <parent link="$(arg summit_prefix)base_chapa"/>
-        <child link="franka_controller_unit_plate"/>
-        <origin xyz="-0.259 0 0.351"/>
-    </joint>
-    <link name="ur_controller_unit_plate">
-        <visual>
-            <geometry>
-                <mesh filename="package://iliad/meshes/ur_controller_box_plate.stl"/>
-            </geometry>
-            <origin rpy="0 0 0" xyz="-0.0175 -0.19 0"/>
-            <material name="grey">
-                <color rgba="1 1 1 1"/>
-            </material>
-        </visual>
-        <collision>
-            <geometry>
-                <mesh filename="package://iliad/meshes/ur_controller_box_plate.stl"/>
-            </geometry>
-            <origin rpy="0 0 0" xyz="-0.0175 -0.19 0"/>
-        </collision>
-        <inertial>
-            <mass value="0"/>
-            <inertia ixx="0.0" ixy="0.0" ixz="0.0" iyy="0.0" iyz="0.0" izz="0.0"/>
-        </inertial>
-    </link>
-    <joint name="controller_unit_TO_ur_plate" type="fixed">
-        <parent link="$(arg summit_prefix)base_chapa"/>
-        <child link="ur_controller_unit_plate"/>
-        <origin xyz="-0.1305 0 0.164"/>
-    </joint>
-    <material name="steel">
-        <color rgba="0 0 0 1.0"/> <!-- rviz green color -->
-    </material>
-    <link name="arms_base">
-        <visual>
-            <geometry>
-                <mesh filename="package://iliad/meshes/arm_base.stl"/>
-            </geometry>
-            <material name="steel"/>
-        </visual>
-        <collision>
-            <geometry>
-                <mesh filename="package://iliad/meshes/arm_base.stl"/>
-            </geometry>
-        </collision>
-        <inertial>
-            <mass value="2"/>   <!-- -->
-            <inertia ixx="0.2741" ixy="0.0" ixz="0.0" iyy="0.125" iyz="0.0" izz="0.2741"/>
-        </inertial>
-    </link>
-    <gazebo reference="arms_base">
-        <material>Gazebo/Grey</material>
-    </gazebo>
-    <gazebo reference="controller_unit">
-        <material>Gazebo/Grey</material>
-    </gazebo>
-    <!---->
-    <gazebo reference="franka_controller_unit_plate">
-        <material>Gazebo/Black</material>
-    </gazebo>
-    <gazebo reference="ur_controller_unit_plate">
-        <material>Gazebo/Black</material>
-    </gazebo>
-    <joint name="summit_to_arms_base" type="fixed">
-        <parent link="$(arg summit_prefix)base_chapa"/>
-        <child link="arms_base"/>
-        <origin xyz="0.135 0.410 0" rpy="0 0 -1.57079632679"/>
-    </joint>
-     <!--********************************************************************************************************************************************* -->
+    <!--********************************************************************************************************************************************* -->
     <!-- ROS Plugins -->
     <gazebo>

File: iliad/urdf/iliad3.urdf.xacro (robot description, xacro)
@@ -1,9 +1,10 @@
 <?xml version="1.0"?>
 <robot name="iliad" xmlns:xacro="http://wiki.ros.org/xacro">
+<!-- Velvet
 <xacro:property name="box_x" value="0.14"/>
 <xacro:property name="box_y" value="0.08"/>
 <xacro:property name="box_z" value="0.28"/>
 <xacro:property name="box_dim" value="${box_x} ${box_y} ${box_z}"/>
-<xacro:property name="mass" value="2"/>
+<xacro:property name="mass" value="1"/>
   <link name="velvet_link">
     <visual>
@@ -26,5 +27,4 @@
   </link>
   <gazebo reference="velvet_link">
-     <!--<static>true</static> -->
     <mu1 value="1.0"/>
     <mu2 value="1.0"/>
@@ -41,3 +41,100 @@
     </collision>
   </gazebo>
+  -->
+<!-- flange
+    <xacro:include filename="$(find iliad)/urdf/flange.urdf.xacro"/>
+    <xacro:property name="fl_box_x" value="0.10"/>
+    <xacro:property name="fl_box_y" value="0.06"/>
+    <xacro:property name="fl_box_z" value="0.08"/>
+    <xacro:property name="fl_box_dim" value="${fl_box_x} ${fl_box_y} ${fl_box_z}"/>
+    <xacro:property name="fl_mass" value="0.300"/>
+    <link name="flange">
+        <visual>
+            <geometry>
+                <box size="${fl_box_dim}"/>
+            </geometry>
+            <origin rpy="0 0 0" xyz="0.02 0 0"/>
+            <material name="grey">
+                <color rgba="0.5 0.5 0.5 1"/>
+            </material>
+        </visual>
+        <collision>
+            <geometry>
+                <box size="${fl_box_dim}"/>
+            </geometry>
+            <origin rpy="0 0 0" xyz="0.02 0 0"/>
+        </collision>
+        <inertial>
+            <mass value="${fl_mass}"/>
+            <inertia ixx="${fl_mass/12*(fl_box_y*fl_box_y+fl_box_z*fl_box_z)}" ixy="0.0" ixz="0.0" iyy="${fl_mass/12*(fl_box_x*fl_box_x+fl_box_z*fl_box_z)}" iyz="0.0" izz="${fl_mass/12*(fl_box_x*fl_box_x+fl_box_y*fl_box_y)}"/>
+            <origin rpy="0 0 0" xyz="0.02 0 0"/>
+        </inertial>
+    </link>
+    <gazebo reference="flange">
+        <material>Gazebo/Grey</material>
+    </gazebo>
+    -->
+    <!-- controller_unit
+    <xacro:property name="ctr_box_x" value="0.25"/>
+    <xacro:property name="ctr_box_y" value="0.46"/>
+    <xacro:property name="ctr_box_z" value="0.25"/>
+    <xacro:property name="ctr_box_dim" value="${ctr_box_x} ${ctr_box_y} ${ctr_box_z}"/>
+    <xacro:property name="ctr_mass" value="12"/>
+        <link name="controller_unit">
+            <visual>
+                <geometry>
+                    <mesh filename="package://iliad/meshes/controller_boxes.stl"/>
+                </geometry>
+                <origin rpy="0 0 0" xyz="-0.1715 -0.2415 0"/>
+                <material name="grey">
+                    <color rgba="0.5 0.5 0.5 1"/>
+                </material>
+            </visual>
+            <collision>
+                <geometry>
+                    <mesh filename="package://iliad/meshes/controller_boxes.stl"/>
+                </geometry>
+                <origin rpy="0 0 0" xyz="-0.1715 -0.2415 0"/>
+            </collision>
+            <inertial>
+                <mass value="${ctr_mass}"/>
+                <inertia ixx="${ctr_mass/12*(ctr_box_y*ctr_box_y+ctr_box_z*ctr_box_z)}" ixy="0.0" ixz="0.0" iyy="${ctr_mass/12*(ctr_box_x*ctr_box_x+ctr_box_z*ctr_box_z)}" iyz="0.0" izz="${ctr_mass/12*(ctr_box_x*ctr_box_x+ctr_box_y*ctr_box_y)}"/>
+                <origin rpy="0 0 0" xyz="0 0 0.13"/>
+            </inertial>
+        </link>
+        <gazebo reference="controller_unit">
+            <material>Gazebo/Grey</material>
+        </gazebo>
+-->
+<!-- arms_base-->
+    <xacro:property name="arb_box_x" value="0.2"/>
+    <xacro:property name="arb_box_y" value="0.57"/>
+    <xacro:property name="arb_box_z" value="0.1"/>
+    <xacro:property name="arb_box_dim" value="${arb_box_x} ${arb_box_y} ${arb_box_z}"/>
+    <xacro:property name="arb_mass" value="2"/>
+    <link name="arms_base">
+        <visual>
+            <geometry>
+                <mesh filename="package://iliad/meshes/arm_base.stl"/>
+            </geometry>
+            <origin xyz="-0.135 0.410 0" rpy="0 0 -1.57079632679"/>
+            <material name="grey">
+                <color rgba="0.5 0.5 0.5 1"/>
+            </material>
+        </visual>
+        <collision>
+            <geometry>
+                <mesh filename="package://iliad/meshes/arm_base.stl"/>
+            </geometry>
+            <origin xyz="-0.135 0.410 0" rpy="0 0 -1.57079632679"/>
+        </collision>
+        <inertial>
+            <mass value="${arb_mass}"/>
+            <inertia ixx="${arb_mass/12*(arb_box_y*arb_box_y+arb_box_z*arb_box_z)}" ixy="0.0" ixz="0.0" iyy="${arb_mass/12*(arb_box_x*arb_box_x+arb_box_z*arb_box_z)}" iyz="0.0" izz="${arb_mass/12*(arb_box_x*arb_box_x+arb_box_y*arb_box_y)}"/>
+            <origin xyz="0 0 0.05" rpy="0 0 0"/>
+        </inertial>
+    </link>
+    <gazebo reference="arms_base">
+        <material>Gazebo/Grey</material>
+    </gazebo>
 </robot>

File: iliad/urdf/velvet_new.urdf.xacro (robot description, xacro)
@@ -1,36 +1,37 @@
 <?xml version="1.0"?>
 <robot xmlns:xacro="http://www.ros.org/wiki/xacro">
-<xacro:property name="box_x" value="0.14"/>
-<xacro:property name="box_y" value="0.08"/>
-<xacro:property name="box_z" value="0.28"/>
-<xacro:property name="box_dim" value="${box_x} ${box_y} ${box_z}"/>
-<xacro:property name="mass" value="2"/>
-<xacro:property name="velvet_mass" value="${100*gr_to_Kg}"/>
-<xacro:macro name="model_velvet" params="parent name *origin">
-    <joint name="${parent}_${name}_base_joint" type="fixed">
+<xacro:property name="vel_box_x" value="0.14"/>
+<xacro:property name="vel_box_y" value="0.08"/>
+<xacro:property name="vel_box_z" value="0.28"/>
+<xacro:property name="vel_box_dim" value="${vel_box_x} ${vel_box_y} ${vel_box_z}"/>
+<xacro:property name="vel_mass" value="1"/>
+<xacro:macro name="velvet_macro" params="parent name *origin">
+    <joint name="${parent}_${name}" type="fixed">
         <xacro:insert_block name="origin"/>
         <parent link="${parent}"/>
-        <child link="${name}_link"/>
+        <child link="${name}"/>
     </joint>
-    <link name="${name}_link">
+    <link name="${name}">
         <visual>
       <geometry>
         <mesh filename="package://iliad/meshes/gazebo_assieme.stl"/>
       </geometry>
-      <color rgba="1.0 0.0 0.0 1.0"/>
+      <material name="green">
+          <color rgba="0 1 0 1"/>
+      </material>
     </visual>
     <inertial>
         <origin xyz="0 0 0"/>
-        <mass value="${mass}"/>
-        <inertia ixx="${mass/12*(box_y*box_y+box_z*box_z)}" ixy="0.0" ixz="0.0" iyy="${mass/12*(box_x*box_x+box_z*box_z)}" iyz="0.0" izz="${mass/12*(box_x*box_x+box_y*box_y)}"/>
+        <mass value="${vel_mass}"/>
+        <inertia ixx="${vel_mass/12*(vel_box_y*vel_box_y+vel_box_z*vel_box_z)}" ixy="0.0" ixz="0.0" iyy="${vel_mass/12*(vel_box_x*vel_box_x+vel_box_z*vel_box_z)}" iyz="0.0" izz="${vel_mass/12*(vel_box_x*vel_box_x+vel_box_y*vel_box_y)}"/>
     </inertial>
     <collision>
       <geometry>
-           <box size="${box_dim}"/>
+           <box size="${vel_box_dim}"/>
       </geometry>
       <origin rpy="0 0 0" xyz="0 0 0"/>
     </collision>
     </link>
-  <gazebo reference="${name}_link">
+  <gazebo reference="${name}">
      <!--<static>true</static> -->
     <mu1 value="1.0"/>

Commit message: prepare to experiments...

File: iliad/urdf/iliad.urdf.xacro (robot description, xacro)
@@ -50,5 +50,5 @@
     </joint>
     <xacro:velvet_macro parent="ur10e_tool0" name="velvet">
-        <origin xyz="0 0 0.14" rpy="0 0 0"/>
+        <origin xyz="0 0.07 0.14" rpy="-0.5326 0 0"/>
     </xacro:velvet_macro>
     <xacro:franka_robot arm_id="$(arg panda_prefix)" joint_limits="${xacro.load_yaml('$(find iliad)/robots/joint_limits.yaml')}"/>
